File: soilmoisture.kicad_pcb (KiCad board)
At the start: 2 copper layers, 33 x 115.6 mm, 9 parts, among them J1 Conn_ARM_JTAG_SWD_10, U1 BT840, U2 BAT-HLD-001, Y1 32KHZ

Commit message: Add co-planar cap fills
Routing:
- net GND: track 35.1 -> 212.1 mm
- net /SOIL_READ: track 23.3 -> 165.3 mm, vias 0 -> 1
- net +BATT: track 41.2 -> 42.7 mm
- net Net-(J1-Pad9): track 0.62 -> 0.00 mm
- added copper zone on B.Cu, net /SOIL_READ
- added copper zone on F.Cu, net /SOIL_READ
- added copper zone on B.Cu, net GND
- added copper zone on F.Cu, net GND
Other:
- board size 33 x 115.6 mm -> 33 x 99.1 mm

Commit message: Add ground plane
Routing:
- net GND: track 212.1 -> 236.0 mm
Changed lines of the file:
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@@
     (thickness 1.6)
     (drawings 8)
-    (tracks 149)
+    (tracks 152)
     (zones 0)
     (modules 9)
@@
   (segment (start 151.13 111.76) (end 151.13 121.92) (width 0.25) (layer F.Cu) (net 55))
   (segment (start 151.13 121.92) (end 151.13 127) (width 0.25) (layer F.Cu) (net 55))
-  (via (at 151.13 67.31) (size 0.8) (drill 0.4) (layers F.Cu B.Cu) (net 55))
   (segment (start 151.13 67.31) (end 151.13 74.93) (width 0.25) (layer B.Cu) (net 55))
   (segment (start 151.13 74.93) (end 151.13 81.28) (width 0.25) (layer B.Cu) (net 55))
@@
   (segment (start 151.13 111.76) (end 151.13 120.65) (width 0.25) (layer B.Cu) (net 55))
   (segment (start 151.13 120.65) (end 151.13 127) (width 0.25) (layer B.Cu) (net 55))
+  (via (at 129.54 66.04) (size 0.8) (drill 0.4) (layers F.Cu B.Cu) (net 55))
+  (segment (start 129.54 66.04) (end 149.86 66.04) (width 0.25) (layer B.Cu) (net 55))
+  (segment (start 149.86 66.04) (end 151.13 67.31) (width 0.25) (layer B.Cu) (net 55))
+  (segment (start 129.54 66.04) (end 128.27 64.77) (width 0.25) (layer B.Cu) (net 55))
   (segment (start 144.07383 45.81144) (end 147.638205 49.375815) (width 0.25) (layer F.Cu) (net 56))
   (segment (start 143.53794 45.81144) (end 144.07383 45.81144) (width 0.25) (layer F.Cu) (net 56))
@@
       )
     )
+  )
+  (zone (net 55) (net_name GND) (layer B.Cu) (hatch edge 0.508)
+    (connect_pads (clearance 0.508))
+    (min_thickness 0.254)
+    (fill yes (arc_segments 16) (thermal_gap 0.508) (thermal_bridge_width 0.508))
+    (polygon
+      (pts
+        (xy 119.38 43.18) (xy 152.4 43.18) (xy 152.4 64.77) (xy 119.38 64.77)
+      )
+    )

Commit message: Update README, fixup ground fill
Routing:
- net GND: track 236.0 -> 224.5 mm, vias 4 -> 5
Changed lines of the file:
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@@
     (thickness 1.6)
     (drawings 8)
-    (tracks 152)
+    (tracks 150)
     (zones 0)
     (modules 9)
@@
   (segment (start 132.08 50.8) (end 135.89 54.61) (width 0.25) (layer B.Cu) (net 55))
   (segment (start 125.73 50.8) (end 132.08 50.8) (width 0.25) (layer B.Cu) (net 55))
-  (segment (start 123.19 50.8) (end 125.73 50.8) (width 0.25) (layer F.Cu) (net 55))
-  (segment (start 121.92 49.53) (end 123.19 50.8) (width 0.25) (layer F.Cu) (net 55))
-  (segment (start 121.92 45.72) (end 121.92 49.53) (width 0.25) (layer F.Cu) (net 55))
-  (segment (start 123.19 44.45) (end 121.92 45.72) (width 0.25) (layer F.Cu) (net 55))
-  (segment (start 127 44.9325) (end 126.5175 44.45) (width 0.25) (layer F.Cu) (net 55))
-  (segment (start 126.5175 44.45) (end 123.19 44.45) (width 0.25) (layer F.Cu) (net 55))
   (segment (start 127.7875 62.23) (end 127.7875 64.2875) (width 0.25) (layer F.Cu) (net 55))
   (segment (start 127.7875 64.2875) (end 129.54 66.04) (width 0.25) (layer F.Cu) (net 55))
@@
   (segment (start 149.86 66.04) (end 151.13 67.31) (width 0.25) (layer B.Cu) (net 55))
   (segment (start 129.54 66.04) (end 128.27 64.77) (width 0.25) (layer B.Cu) (net 55))
+  (segment (start 140.91774 44.61002) (end 141.07776 44.45) (width 0.25) (layer F.Cu) (net 55))
+  (segment (start 139.91844 44.61002) (end 140.91774 44.61002) (width 0.25) (layer F.Cu) (net 55))
+  (via (at 142.24 44.45) (size 0.8) (drill 0.4) (layers F.Cu B.Cu) (net 55))
+  (segment (start 141.07776 44.45) (end 142.24 44.45) (width 0.25) (layer F.Cu) (net 55))
   (segment (start 144.07383 45.81144) (end 147.638205 49.375815) (width 0.25) (layer F.Cu) (net 56))
   (segment (start 143.53794 45.81144) (end 144.07383 45.81144) (width 0.25) (layer F.Cu) (net 56))
@@
   (segment (start 133.94 55.29) (end 133.94 57.15) (width 0.25) (layer F.Cu) (net 59))
   (segment (start 134.62 54.61) (end 133.94 55.29) (width 0.25) (layer F.Cu) (net 59))
-  (segment (start 142.03807 54.61) (end 134.62 54.61) (width 0.25) (layer F.Cu) (net 59))
   (segment (start 143.53794 53.51018) (end 143.13789 53.51018) (width 0.25) (layer F.Cu) (net 59))
   (segment (start 143.13789 53.51018) (end 142.03807 54.61) (width 0.25) (layer F.Cu) (net 59))
+  (segment (start 142.03807 54.61) (end 134.62 54.61) (width 0.25) (layer F.Cu) (net 59))
   (segment (start 141.78788 51.41214) (end 141.78788 49.98212) (width 0.25) (layer F.Cu) (net 60))
   (segment (start 141.78788 49.98212) (end 141.78788 45.72) (width 0.25) (layer F.Cu) (net 60))
